File: subsch/DBUS.kicad_sch (KiCad schematic)
At the start: 5 parts

Commit message: USB2UART
Parts:
- C25: value (none) -> 100n; footprint (none) -> Capacitor_SMD:C_0603_1608Metric
- Q1: value (none) -> S8050; footprint (none) -> Package_TO_SOT_SMD:SOT-23
- R11: value (none) -> 4.7K; footprint (none) -> Resistor_SMD:R_0603_1608Metric
- R12: value (none) -> 47K; footprint (none) -> Resistor_SMD:R_0603_1608Metric
- U8: value (none) -> CH340E; footprint (none) -> Package_SO:MSOP-10_3x3mm_P0.5mm
Changed lines of the file:
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@@
       (effects (font (size 1.27 1.27)) (justify right))
     )
-    (property "Value" "" (id 1) (at 108.712 89.916 0)
+    (property "Value" "100n" (id 1) (at 108.712 89.916 0)
       (effects (font (size 1.27 1.27)) (justify right))
     )
-    (property "Footprint" "" (id 2) (at 107.696 87.376 0)
+    (property "Footprint" "Capacitor_SMD:C_0603_1608Metric" (id 2) (at 107.696 87.376 0)
       (effects (font (size 1.27 1.27)) hide)
     )
@@
       (effects (font (size 1.27 1.27)) hide)
     )
-    (property "Value" "" (id 1) (at 160.782 110.7345 0))
+    (property "Value" "GND" (id 1) (at 160.782 110.7345 0))
     (property "Footprint" "" (id 2) (at 160.782 106.172 0)
       (effects (font (size 1.27 1.27)) hide)
@@
       (effects (font (size 1.27 1.27)) hide)
     )
-    (property "Value" "" (id 1) (at 130.302 68.0235 0))
+    (property "Value" "VCC" (id 1) (at 130.302 68.0235 0))
     (property "Footprint" "" (id 2) (at 130.302 71.628 0)
       (effects (font (size 1.27 1.27)) hide)
@@
       (effects (font (size 1.27 1.27)) (justify left))
     )
-    (property "Value" "" (id 1) (at 153.8986 79.5906 0)
+    (property "Value" "4.7K" (id 1) (at 153.8986 79.5906 0)
       (effects (font (size 1.27 1.27)) (justify left))
     )
-    (property "Footprint" "" (id 2) (at 152.4 77.724 0)
+    (property "Footprint" "Resistor_SMD:R_0603_1608Metric" (id 2) (at 152.4 77.724 0)
       (effects (font (size 1.27 1.27)) hide)
     )
@@
       (effects (font (size 1.27 1.27)) (justify left))
     )
-    (property "Value" "" (id 1) (at 134.8614 107.0326 0)
+    (property "Value" "CH340E" (id 1) (at 134.8614 107.0326 0)
       (effects (font (size 1.27 1.27)) (justify left))
     )
-    (property "Footprint" "" (id 2) (at 134.112 103.378 0)
+    (property "Footprint" "Package_SO:MSOP-10_3x3mm_P0.5mm" (id 2) (at 134.112 103.378 0)
       (effects (font (size 1.27 1.27)) (justify left) hide)
     )
@@
       (effects (font (size 1.27 1.27)) (justify left))
     )
-    (property "Value" "" (id 1) (at 162.2806 100.6726 0)
+    (property "Value" "47K" (id 1) (at 162.2806 100.6726 0)
       (effects (font (size 1.27 1.27)) (justify left))
     )
-    (property "Footprint" "" (id 2) (at 160.782 98.806 0)
+    (property "Footprint" "Resistor_SMD:R_0603_1608Metric" (id 2) (at 160.782 98.806 0)
       (effects (font (size 1.27 1.27)) hide)
     )
@@
       (effects (font (size 1.27 1.27)) hide)
     )
-    (property "Value" "" (id 1) (at 132.842 110.7345 0))
+    (property "Value" "GND" (id 1) (at 132.842 110.7345 0))
     (property "Footprint" "" (id 2) (at 132.842 106.172 0)
       (effects (font (size 1.27 1.27)) hide)
@@
       (effects (font (size 1.27 1.27)) hide)
     )
-    (property "Value" "" (id 1) (at 107.696 96.5105 0))
+    (property "Value" "GND" (id 1) (at 107.696 96.5105 0))
     (property "Footprint" "" (id 2) (at 107.696 91.948 0)
       (effects (font (size 1.27 1.27)) hide)
@@
       (effects (font (size 1.27 1.27)) hide)
     )
-    (property "Value" "" (id 1) (at 107.696 79.7075 0))
+    (property "Value" "VCC" (id 1) (at 107.696 79.7075 0))
     (property "Footprint" "" (id 2) (at 107.696 83.312 0)
       (effects (font (size 1.27 1.27)) hide)
@@
       (effects (font (size 1.27 1.27)) hide)
     )
-    (property "Value" "" (id 1) (at 152.4 67.5155 0))
+    (property "Value" "VCC" (id 1) (at 152.4 67.5155 0))
     (property "Footprint" "" (id 2) (at 152.4 71.12 0)
       (effects (font (size 1.27 1.27)) hide)
@@
       (effects (font (size 1.27 1.27)) (justify left))
     )
-    (property "Value" "" (id 1) (at 150.0886 95.0846 0)
+    (property "Value" "S8050" (id 1) (at 150.0886 95.0846 0)
       (effects (font (size 1.27 1.27)) (justify left))
     )
-    (property "Footprint" "" (id 2) (at 149.86 90.678 0)
+    (property "Footprint" "Package_TO_SOT_SMD:SOT-23" (id 2) (at 149.86 90.678 0)
       (effects (font (size 1.27 1.27)) hide)
     )
@@
       (effects (font (size 1.27 1.27)) hide)
     )
-    (property "Value" "" (id 1) (at 152.4 110.7345 0))
+    (property "Value" "GND" (id 1) (at 152.4 110.7345 0))
     (property "Footprint" "" (id 2) (at 152.4 106.172 0)
       (effects (font (size 1.27 1.27)) hide)
