File: subsch/USB_HUB.kicad_sch (KiCad schematic)
At the start: 7 parts

Commit message: USB2UART
Parts:
- C19, C20: value (none) -> 10u; footprint (none) -> Capacitor_SMD:C_0603_1608Metric
- C21, C22: value (none) -> 18p; footprint (none) -> Capacitor_SMD:C_0603_1608Metric
- C23: value (none) -> 100n; footprint (none) -> Capacitor_SMD:C_0603_1608Metric
- U6: value (none) -> SL2.1S; footprint (none) -> MyLib:SL2.1S-SSOP-16
- Y1: value (none) -> 12M; footprint (none) -> Crystal:Crystal_SMD_3225-4Pin_3.2x2.5mm
Changed lines of the file:
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@@
       (effects (font (size 1.27 1.27)) hide)
     )
-    (property "Value" "" (id 1) (at 128.651 51.787 90)
+    (property "Value" "GND" (id 1) (at 128.651 51.787 90)
       (effects (font (size 1.27 1.27)) (justify right))
     )
@@
       (effects (font (size 1.27 1.27)) hide)
     )
-    (property "Value" "" (id 1) (at 128.651 55.343 90)
+    (property "Value" "GND" (id 1) (at 128.651 55.343 90)
       (effects (font (size 1.27 1.27)) (justify right))
     )
@@
     (in_bom yes) (on_board yes)
     (property "Reference" "C22" (id 0) (at 87.376 67.945 90))
-    (property "Value" "" (id 1) (at 93.218 67.691 90))
-    (property "Footprint" "" (id 2) (at 89.916 66.548 0)
+    (property "Value" "18p" (id 1) (at 93.218 67.691 90))
+    (property "Footprint" "Capacitor_SMD:C_0603_1608Metric" (id 2) (at 89.916 66.548 0)
       (effects (font (size 1.27 1.27)) hide)
     )
@@
       (effects (font (size 1.27 1.27)) (justify left))
     )
-    (property "Value" "" (id 1) (at 117.3354 88.1858 0)
-      (effects (font (size 1.27 1.27)) (justify left))
-    )
-    (property "Footprint" "" (id 2) (at 116.078 57.785 0)
+    (property "Value" "SL2.1S" (id 1) (at 117.3354 88.1858 0)
+      (effects (font (size 1.27 1.27)) (justify left))
+    )
+    (property "Footprint" "MyLib:SL2.1S-SSOP-16" (id 2) (at 116.078 57.785 0)
       (effects (font (size 1.27 1.27)) hide)
     )
@@
       (effects (font (size 1.27 1.27)) (justify left))
     )
-    (property "Value" "" (id 1) (at 87.884 84.328 0)
-      (effects (font (size 1.27 1.27)) (justify right))
-    )
-    (property "Footprint" "" (id 2) (at 88.392 82.804 0)
+    (property "Value" "100n" (id 1) (at 87.884 84.328 0)
+      (effects (font (size 1.27 1.27)) (justify right))
+    )
+    (property "Footprint" "Capacitor_SMD:C_0603_1608Metric" (id 2) (at 88.392 82.804 0)
       (effects (font (size 1.27 1.27)) hide)
     )
@@
     (in_bom yes) (on_board yes)
     (property "Reference" "C19" (id 0) (at 118.237 50.165 90))
-    (property "Value" "" (id 1) (at 122.809 50.165 90))
-    (property "Footprint" "" (id 2) (at 120.396 51.308 0)
+    (property "Value" "10u" (id 1) (at 122.809 50.165 90))
+    (property "Footprint" "Capacitor_SMD:C_0603_1608Metric" (id 2) (at 120.396 51.308 0)
       (effects (font (size 1.27 1.27)) hide)
     )
@@
       (effects (font (size 1.27 1.27)) hide)
     )
-    (property "Value" "" (id 1) (at 81.28 66.5385 0))
+    (property "Value" "GND" (id 1) (at 81.28 66.5385 0))
     (property "Footprint" "" (id 2) (at 81.28 61.976 0)
       (effects (font (size 1.27 1.27)) hide)
@@
       (effects (font (size 1.27 1.27)) hide)
     )
-    (property "Value" "" (id 1) (at 88.392 91.9385 0))
+    (property "Value" "GND" (id 1) (at 88.392 91.9385 0))
     (property "Footprint" "" (id 2) (at 88.392 87.376 0)
       (effects (font (size 1.27 1.27)) hide)
@@
       (effects (font (size 1.27 1.27)) hide)
     )
-    (property "Value" "" (id 1) (at 110.236 47.1955 0))
+    (property "Value" "+5V" (id 1) (at 110.236 47.1955 0))
     (property "Footprint" "" (id 2) (at 110.236 50.8 0)
       (effects (font (size 1.27 1.27)) hide)
@@
       (effects (font (size 1.27 1.27)) hide)
     )
-    (property "Value" "" (id 1) (at 88.392 76.1515 0))
+    (property "Value" "+5V" (id 1) (at 88.392 76.1515 0))
     (property "Footprint" "" (id 2) (at 88.392 79.756 0)
       (effects (font (size 1.27 1.27)) hide)
@@
       (effects (font (size 1.27 1.27)) (justify left))
     )
-    (property "Value" "" (id 1) (at 80.772 60.452 0)
-      (effects (font (size 1.27 1.27)) (justify right))
-    )
-    (property "Footprint" "" (id 2) (at 81.28 58.928 0)
+    (property "Value" "18p" (id 1) (at 80.772 60.452 0)
+      (effects (font (size 1.27 1.27)) (justify right))
+    )
+    (property "Footprint" "Capacitor_SMD:C_0603_1608Metric" (id 2) (at 81.28 58.928 0)
       (effects (font (size 1.27 1.27)) hide)
     )
@@
     (in_bom yes) (on_board yes)
     (property "Reference" "C20" (id 0) (at 118.237 53.721 90))
-    (property "Value" "" (id 1) (at 122.809 53.721 90))
-    (property "Footprint" "" (id 2) (at 120.396 54.864 0)
+    (property "Value" "10u" (id 1) (at 122.809 53.721 90))
+    (property "Footprint" "Capacitor_SMD:C_0603_1608Metric" (id 2) (at 120.396 54.864 0)
       (effects (font (size 1.27 1.27)) hide)
     )
@@
       (effects (font (size 1.27 1.27)) hide)
     )
-    (property "Value" "" (id 1) (at 96.647 61.947 90)
+    (property "Value" "GND" (id 1) (at 96.647 61.947 90)
       (effects (font (size 1.27 1.27)) (justify right))
     )
@@
       (effects (font (size 1.27 1.27)) hide)
     )
-    (property "Value" "" (id 1) (at 115.316 92.7005 0))
+    (property "Value" "GND" (id 1) (at 115.316 92.7005 0))
     (property "Footprint" "" (id 2) (at 115.316 88.138 0)
       (effects (font (size 1.27 1.27)) hide)
@@
     (in_bom yes) (on_board yes)
     (property "Reference" "Y1" (id 0) (at 89.154 55.626 90))
-    (property "Value" "" (id 1) (at 89.662 57.912 90))
-    (property "Footprint" "" (id 2) (at 87.376 61.468 0)
-      (effects (font (size 1.27 1.27)) hide)
-    )
+    (property "Value" "12M" (id 1) (at 89.662 57.912 90))
+    (property "Footprint" "Crystal:Crystal_SMD_3225-4Pin_3.2x2.5mm" (id 2) (at 87.376 61.468 0)
+      (effects (font (size 1.27 1.27)) hide)
+    )
