File: USB2UART.kicad_pcb (KiCad board)
At the start: 2 copper layers, 43.9 x 34.3 mm, 33 parts, among them J1 Conn_01x04, J2 Conn_01x03, J3 Conn_01x03, J4 Conn_01x03, J5 Conn_01x03, Q1 S8050, U3 HX9193, U6 SL2.1S, U7 CH340E, U8 CH340E, Y1 12M

Commit message: small changes
Parts:
- moved C25 2.57 mm to (109.7, 83.1), turned to 180 degrees
- moved C27 0.83 mm to (113.0, 83.1), turned to 180 degrees
Routing:
- net /UART1/TXD: track 13.2 -> 10.2 mm
- net +5V: track 92.4 -> 90.5 mm
Other:
- board text added: "USB2UART"
- board text removed: "USB2XXX"

Commit message: another right version
Parts:
- J4, J5: value Conn_01x03 -> Conn_01x04
Changed lines of the file:
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@@
     (descr "Molex CLIK-Mate series connector, 502386-0470 (http://www.molex.com/pdm_docs/sd/5023860270_sd.pdf), generated with kicad-footprint-generator")
     (tags "connector Molex CLIK-Mate top entry")
-    (property "Sheetfile" "USB2XXX.kicad_sch")
+    (property "Sheetfile" "USB2UART.kicad_sch")
     (property "Sheetname" "")
     (attr smd)
@@
     (descr "JST GH series connector, SM04B-GHS-TB (http://www.jst-mfg.com/product/pdf/eng/eGH.pdf), generated with kicad-footprint-generator")
     (tags "connector JST GH top entry")
-    (property "Sheetfile" "USB2XXX.kicad_sch")
+    (property "Sheetfile" "USB2UART.kicad_sch")
     (property "Sheetname" "")
     (attr smd)
@@
       (effects (font (size 1 1) (thickness 0.15)))
     )
-    (fp_text value "Conn_01x03" (at 0 3.9) (layer "F.Fab")
+    (fp_text value "Conn_01x04" (at 0 3.9) (layer "F.Fab")
       (effects (font (size 1 1) (thickness 0.15)))
     )
@@
     (descr "Capacitor SMD 0603 (1608 Metric), square (rectangular) end terminal, IPC_7351 nominal, (Body size source: IPC-SM-782 page 76, https://www.pcb-3d.com/wordpress/wp-content/uploads/ipc-sm-782a_amendment_1_and_2.pdf), generated with kicad-footprint-generator")
     (tags "capacitor")
-    (property "Sheetfile" "USB2XXX.kicad_sch")
+    (property "Sheetfile" "USB2UART.kicad_sch")
     (property "Sheetname" "")
     (attr smd)
@@
     (descr "Capacitor SMD 0603 (1608 Metric), square (rectangular) end terminal, IPC_7351 nominal, (Body size source: IPC-SM-782 page 76, https://www.pcb-3d.com/wordpress/wp-content/uploads/ipc-sm-782a_amendment_1_and_2.pdf), generated with kicad-footprint-generator")
     (tags "capacitor")
-    (property "Sheetfile" "USB2XXX.kicad_sch")
+    (property "Sheetfile" "USB2UART.kicad_sch")
     (property "Sheetname" "")
     (attr smd)
@@
     (descr "SOD-323")
     (tags "SOD-323")
-    (property "Sheetfile" "USB2XXX.kicad_sch")
+    (property "Sheetfile" "USB2UART.kicad_sch")
     (property "Sheetname" "")
     (attr smd)
@@
     (descr "JST GH series connector, SM04B-GHS-TB (http://www.jst-mfg.com/product/pdf/eng/eGH.pdf), generated with kicad-footprint-generator")
     (tags "connector JST GH top entry")
-    (property "Sheetfile" "USB2XXX.kicad_sch")
+    (property "Sheetfile" "USB2UART.kicad_sch")
     (property "Sheetname" "")
     (attr smd)
@@
       (effects (font (size 1 1) (thickness 0.15)))
     )
-    (fp_text value "Conn_01x03" (at 0 3.9) (layer "F.Fab")
+    (fp_text value "Conn_01x04" (at 0 3.9) (layer "F.Fab")
       (effects (font (size 1 1) (thickness 0.15)))
     )
@@
     (descr "SOD-323")
     (tags "SOD-323")
-    (property "Sheetfile" "USB2XXX.kicad_sch")
+    (property "Sheetfile" "USB2UART.kicad_sch")
     (property "Sheetname" "")
     (attr smd)
@@
     (descr "JST GH series connector, SM03B-GHS-TB (http://www.jst-mfg.com/product/pdf/eng/eGH.pdf), generated with kicad-footprint-generator")
     (tags "connector JST GH top entry")
-    (property "Sheetfile" "USB2XXX.kicad_sch")
+    (property "Sheetfile" "USB2UART.kicad_sch")
     (property "Sheetname" "")
     (attr smd)
@@
     (descr "SOD-323")
     (tags "SOD-323")
-    (property "Sheetfile" "USB2XXX.kicad_sch")
+    (property "Sheetfile" "USB2UART.kicad_sch")
     (property "Sheetname" "")
     (attr smd)
@@
     (descr "JST GH series connector, SM03B-GHS-TB (http://www.jst-mfg.com/product/pdf/eng/eGH.pdf), generated with kicad-footprint-generator")
     (tags "connector JST GH top entry")
-    (property "Sheetfile" "USB2XXX.kicad_sch")
+    (property "Sheetfile" "USB2UART.kicad_sch")
     (property "Sheetname" "")
     (attr smd)
@@
     (descr "LED SMD 0603 (1608 Metric), square (rectangular) end terminal, IPC_7351 nominal, (Body size source: http://www.tortai-tech.com/upload/download/2011102023233369053.pdf), generated with kicad-footprint-generator")
     (tags "LED")
-    (property "Sheetfile" "USB2XXX.kicad_sch")
+    (property "Sheetfile" "USB2UART.kicad_sch")
     (property "Sheetname" "")
     (attr smd)
@@
     (descr "Resistor SMD 0603 (1608 Metric), square (rectangular) end terminal, IPC_7351 nominal, (Body size source: IPC-SM-782 page 72, https://www.pcb-3d.com/wordpress/wp-content/uploads/ipc-sm-782a_amendment_1_and_2.pdf), generated with kicad-footprint-generator")
     (tags "resistor")
-    (property "Sheetfile" "USB2XXX.kicad_sch")
+    (property "Sheetfile" "USB2UART.kicad_sch")
     (property "Sheetname" "")
     (attr smd)

Commit message: final
Parts:
- moved C1 5.72 mm to (113.4, 65.0)
- moved C10 4.36 mm to (120.1, 68.6), turned to 90 degrees
- moved U1 1.85 mm to (116.7, 68.0), turned to 90 degrees
Routing:
- net /UART1/TXD: track 10.2 -> 4.28 mm, vias 2 -> 0
- net /UART1/RXD: track 9.90 -> 4.59 mm
- net /UART1/D-: track 10.9 -> 12.8 mm
- net +5V: track 90.5 -> 88.6 mm
- net /UART1/D+: track 10.9 -> 12.1 mm
- net VCC: track 106.2 -> 105.3 mm, vias 2 -> 0

Commit message: final
Parts:
- moved C23 23.0 mm to (118.3, 64.3), turned to 0 degrees
- moved C1 1.00 mm to (113.4, 66.0)
- moved C10 1.00 mm to (120.1, 69.6)
- moved U1 1.00 mm to (116.7, 69.0)
Routing:
- net +5V: track 88.6 -> 83.6 mm
- net /UART1/TXD: track 4.28 -> 5.28 mm
- net /UART1/RXD: track 4.59 -> 5.59 mm
- net VCC: track 105.3 -> 104.7 mm
- net /UART1/D-: track 12.8 -> 12.3 mm
- net /UART1/D+: track 12.1 -> 11.5 mm

Commit message: final
Parts:
- moved C9 9.19 mm to (93.5, 72.1)
Routing:
- net +5V: track 83.6 -> 79.7 mm
