File: DBUS.kicad_sch (KiCad schematic)
At the start: 12 parts, among them Q1 S8050, Q2 Q_PNP_BCE, Q3 Q_PNP_BCE, U2 CH340E

Commit message: All 0603 version
Parts:
- C7, C8: footprint Capacitor_SMD:C_0402_1005Metric -> Capacitor_SMD:C_0603_1608Metric
- D5: footprint LED_SMD:LED_0402_1005Metric -> LED_SMD:LED_0603_1608Metric
- R2, R3, R4, R5, R6: footprint Resistor_SMD:R_0402_1005Metric -> Resistor_SMD:R_0603_1608Metric
Changed lines of the file:
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@@
       (effects (font (size 1.27 1.27)) (justify left))
     )
-    (property "Footprint" "Resistor_SMD:R_0402_1005Metric" (at 115.697 82.423 0)
+    (property "Footprint" "Resistor_SMD:R_0603_1608Metric" (at 115.697 82.423 0)
       (effects (font (size 1.27 1.27)) hide)
     )
@@
       (effects (font (size 1.27 1.27)) (justify right))
     )
-    (property "Footprint" "Capacitor_SMD:C_0402_1005Metric" (at 71.247 92.583 0)
+    (property "Footprint" "Capacitor_SMD:C_0603_1608Metric" (at 71.247 92.583 0)
       (effects (font (size 1.27 1.27)) hide)
     )
@@
       (effects (font (size 1.27 1.27)))
     )
-    (property "Footprint" "LED_SMD:LED_0402_1005Metric" (at 211.963 88.773 0)
+    (property "Footprint" "LED_SMD:LED_0603_1608Metric" (at 211.963 88.773 0)
       (effects (font (size 1.27 1.27)) hide)
     )
@@
       (effects (font (size 1.27 1.27)))
     )
-    (property "Footprint" "Resistor_SMD:R_0402_1005Metric" (at 168.783 82.931 90)
+    (property "Footprint" "Resistor_SMD:R_0603_1608Metric" (at 168.783 82.931 90)
       (effects (font (size 1.27 1.27)) hide)
     )
@@
       (effects (font (size 1.27 1.27)) (justify left))
     )
-    (property "Footprint" "Capacitor_SMD:C_0402_1005Metric" (at 158.3182 90.043 0)
+    (property "Footprint" "Capacitor_SMD:C_0603_1608Metric" (at 158.3182 90.043 0)
       (effects (font (size 1.27 1.27)) hide)
     )
@@
       (effects (font (size 1.27 1.27)))
     )
-    (property "Footprint" "Resistor_SMD:R_0402_1005Metric" (at 197.993 90.551 90)
+    (property "Footprint" "Resistor_SMD:R_0603_1608Metric" (at 197.993 90.551 90)
       (effects (font (size 1.27 1.27)) hide)
     )
@@
       (effects (font (size 1.27 1.27)) (justify left))
     )
-    (property "Footprint" "Resistor_SMD:R_0402_1005Metric" (at 124.587 104.013 0)
+    (property "Footprint" "Resistor_SMD:R_0603_1608Metric" (at 124.587 104.013 0)
       (effects (font (size 1.27 1.27)) hide)
     )
@@
       (effects (font (size 1.27 1.27)))
     )
-    (property "Footprint" "Resistor_SMD:R_0402_1005Metric" (at 124.333 88.011 90)
-      (effects (font (size 1.27 1.27)) hide)
-    )
+    (property "Footprint" "Resistor_SMD:R_0603_1608Metric" (at 124.333 88.011 90)
+      (effects (font (size 1.27 1.27)) hide)
+    )
