File: UART.kicad_sch (KiCad schematic)
At the start: 17 parts, among them Q4 Q_PNP_BCE, Q5 Q_PNP_BCE, Q6 Q_PNP_BCE, Q7 Q_PNP_BCE, U3 CH340E, U4 ESDS314

Commit message: All 0603 version
Parts:
- C10, C11, C9: footprint Capacitor_SMD:C_0402_1005Metric -> Capacitor_SMD:C_0603_1608Metric
- D6, D7: footprint LED_SMD:LED_0402_1005Metric -> LED_SMD:LED_0603_1608Metric
- R10, R11, R12, R7, R8, R9: footprint Resistor_SMD:R_0402_1005Metric -> Resistor_SMD:R_0603_1608Metric
Changed lines of the file:
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@@
       (effects (font (size 1.27 1.27)))
     )
-    (property "Footprint" "Resistor_SMD:R_0402_1005Metric" (at 199.644 86.233 90)
+    (property "Footprint" "Resistor_SMD:R_0603_1608Metric" (at 199.644 86.233 90)
       (effects (font (size 1.27 1.27)) hide)
     )
@@
       (effects (font (size 1.27 1.27)))
     )
-    (property "Footprint" "Resistor_SMD:R_0402_1005Metric" (at 199.644 106.553 90)
+    (property "Footprint" "Resistor_SMD:R_0603_1608Metric" (at 199.644 106.553 90)
       (effects (font (size 1.27 1.27)) hide)
     )
@@
       (effects (font (size 1.27 1.27)))
     )
-    (property "Footprint" "Resistor_SMD:R_0402_1005Metric" (at 170.434 98.933 90)
+    (property "Footprint" "Resistor_SMD:R_0603_1608Metric" (at 170.434 98.933 90)
       (effects (font (size 1.27 1.27)) hide)
     )
@@
       (effects (font (size 1.27 1.27)))
     )
-    (property "Footprint" "LED_SMD:LED_0402_1005Metric" (at 213.614 84.455 0)
+    (property "Footprint" "LED_SMD:LED_0603_1608Metric" (at 213.614 84.455 0)
       (effects (font (size 1.27 1.27)) hide)
     )
@@
       (effects (font (size 1.27 1.27)))
     )
-    (property "Footprint" "LED_SMD:LED_0402_1005Metric" (at 213.614 104.775 0)
+    (property "Footprint" "LED_SMD:LED_0603_1608Metric" (at 213.614 104.775 0)
       (effects (font (size 1.27 1.27)) hide)
     )
@@
       (effects (font (size 1.27 1.27)))
     )
-    (property "Footprint" "Resistor_SMD:R_0402_1005Metric" (at 170.434 78.613 90)
+    (property "Footprint" "Resistor_SMD:R_0603_1608Metric" (at 170.434 78.613 90)
       (effects (font (size 1.27 1.27)) hide)
     )
@@
       (effects (font (size 1.27 1.27)) (justify left))
     )
-    (property "Footprint" "Capacitor_SMD:C_0402_1005Metric" (at 159.9692 85.725 0)
+    (property "Footprint" "Capacitor_SMD:C_0603_1608Metric" (at 159.9692 85.725 0)
       (effects (font (size 1.27 1.27)) hide)
     )
@@
       (effects (font (size 1.27 1.27)) (justify right))
     )
-    (property "Footprint" "Capacitor_SMD:C_0402_1005Metric" (at 66.294 89.535 0)
+    (property "Footprint" "Capacitor_SMD:C_0603_1608Metric" (at 66.294 89.535 0)
       (effects (font (size 1.27 1.27)) hide)
     )
@@
       (effects (font (size 1.27 1.27)))
     )
-    (property "Footprint" "Resistor_SMD:R_0402_1005Metric" (at 125.984 83.693 90)
+    (property "Footprint" "Resistor_SMD:R_0603_1608Metric" (at 125.984 83.693 90)
       (effects (font (size 1.27 1.27)) hide)
     )
@@
       (effects (font (size 1.27 1.27)) (justify left))
     )
-    (property "Footprint" "Capacitor_SMD:C_0402_1005Metric" (at 159.9692 106.045 0)
+    (property "Footprint" "Capacitor_SMD:C_0603_1608Metric" (at 159.9692 106.045 0)
       (effects (font (size 1.27 1.27)) hide)
     )
@@
       (effects (font (size 1.27 1.27)))
     )
-    (property "Footprint" "Resistor_SMD:R_0402_1005Metric" (at 125.984 104.013 90)
-      (effects (font (size 1.27 1.27)) hide)
-    )
+    (property "Footprint" "Resistor_SMD:R_0603_1608Metric" (at 125.984 104.013 90)
+      (effects (font (size 1.27 1.27)) hide)
+    )
