File: USB2UART.kicad_sch (KiCad schematic)
At the start: 12 parts, among them J1 Conn_01x03, J2 Conn_01x04, J3 Conn_01x03, U5 HX9193

Commit message: All 0603 version
Parts:
- added D1: GREEN, LED_SMD:LED_0603_1608Metric, symbol Device:LED
- added R4: 1K, Resistor_SMD:R_0603_1608Metric, symbol Device:R_Small
- C12, C13: footprint Capacitor_SMD:C_0402_1005Metric -> Capacitor_SMD:C_0603_1608Metric
Connections:
- net GND: now also D1.1 (K)
- net VCC: now also R4.2
- new net: D1.2 (A), R4.1
Changed lines of the file:
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@@
+    (stroke (width 0) (type default))
+  )
+  (wire (pts (xy 68.834 102.489) (xy 68.834 107.061))
     (stroke (width 0) (type default))
   )
@@
     (stroke (width 0) (type default))
   )
+  (wire (pts (xy 68.834 93.599) (xy 68.834 94.869))
+    (stroke (width 0) (type default))
+  )
   (wire (pts (xy 117.475 83.693) (xy 106.553 83.693))
     (stroke (width 0) (type default))
@@
   )
   (wire (pts (xy 55.626 51.943) (xy 58.166 51.943))
+    (stroke (width 0) (type default))
+  )
+  (wire (pts (xy 68.834 84.709) (xy 68.834 88.519))
     (stroke (width 0) (type default))
   )
@@
       (effects (font (size 1.27 1.27)) (justify right))
     )
-    (property "Footprint" "Capacitor_SMD:C_0402_1005Metric" (at 55.626 54.483 0)
+    (property "Footprint" "Capacitor_SMD:C_0603_1608Metric" (at 55.626 54.483 0)
       (effects (font (size 1.27 1.27)) hide)
     )
@@
     )
   )
+  (symbol (lib_id "Device:LED") (at 68.834 98.679 90) (unit 1)
+    (in_bom yes) (on_board yes) (dnp no)
+    (property "Reference" "D1" (at 64.897 99.06 90)
+      (effects (font (size 1.27 1.27)) (justify right))
+    )
+    (property "Value" "GREEN" (at 67.818 100.203 0)
+      (effects (font (size 1.27 1.27)) (justify right))
+    )
+    (property "Footprint" "LED_SMD:LED_0603_1608Metric" (at 68.834 98.679 0)
+      (effects (font (size 1.27 1.27)) hide)
+    )
+    (property "Datasheet" "~" (at 68.834 98.679 0)
+      (effects (font (size 1.27 1.27)) hide)
+    )
+    (pin "1")
+    (pin "2")
+    (instances
+      (project "EtherCAT_FUNC"
+        (path "/342eefad-8419-4edc-841f-71a31e56750b/e0fc0fcc-c6e0-408f-913f-bc6bd8418cc7"
+          (reference "D1") (unit 1)
+        )
+        (path "/342eefad-8419-4edc-841f-71a31e56750b"
+          (reference "D3") (unit 1)
+        )
+      )
+      (project "USB2UART"
+        (path "/75368248-08b1-4e75-aab1-d4baf4ebc338"
+          (reference "D2") (unit 1)
+        )
+      )
+      (project "EtherCAT2XXX"
+        (path "/8e0527a1-64cc-4c21-af5a-5910f4c387cc/fa5393d6-c3e4-4b31-a507-98a55f9f6a14"
+          (reference "D4") (unit 1)
+        )
+      )
+    )
+  )
   (symbol (lib_id "MyLib:HX9193") (at 68.326 57.023 0) (unit 1)
     (in_bom yes) (on_board yes) (dnp no) (fields_autoplaced)
@@
       (effects (font (size 1.27 1.27)) (justify right))
     )
-    (property "Footprint" "Capacitor_SMD:C_0402_1005Metric" (at 80.518 57.785 0)
+    (property "Footprint" "Capacitor_SMD:C_0603_1608Metric" (at 80.518 57.785 0)
       (effects (font (size 1.27 1.27)) hide)
     )
@@
     )
   )
+  (symbol (lib_id "power:VCC") (at 68.834 84.709 0) (unit 1)
+    (in_bom yes) (on_board yes) (dnp no) (fields_autoplaced)
+    (property "Reference" "#PWR02" (at 68.834 88.519 0)
+      (effects (font (size 1.27 1.27)) hide)
+    )
+    (property "Value" "VCC" (at 68.834 81.1045 0)
+      (effects (font (size 1.27 1.27)))
+    )
+    (property "Footprint" "" (at 68.834 84.709 0)
+      (effects (font (size 1.27 1.27)) hide)
+    )
+    (property "Datasheet" "" (at 68.834 84.709 0)
+      (effects (font (size 1.27 1.27)) hide)
+    )
+    (pin "1")
+    (instances
+      (project "USB2UART"
+        (path "/75368248-08b1-4e75-aab1-d4baf4ebc338"
+          (reference "#PWR02") (unit 1)
+        )
+      )
+      (project "USB2XXX"
+        (path "/e63e39d7-6ac0-4ffd-8aa3-1841a4541b55/4d9859dd-6831-4569-841e-8b44f9c9ad5e"
+          (reference "#PWR035") (unit 1)
+        )
+      )
+    )
+  )
   (symbol (lib_id "power:GND") (at 55.626 63.881 0) (unit 1)
     (in_bom yes) (on_board yes) (dnp no) (fields_autoplaced)
@@
     )
   )
+  (symbol (lib_id "Device:R_Small") (at 68.834 91.059 180) (unit 1)
+    (in_bom yes) (on_board yes) (dnp no)
+    (property "Reference" "R4" (at 69.85 88.773 0)
+      (effects (font (size 1.27 1.27)) (justify right))
+    )
+    (property "Value" "1K" (at 70.104 92.329 0)
+      (effects (font (size 1.27 1.27)) (justify right))
+    )
+    (property "Footprint" "Resistor_SMD:R_0603_1608Metric" (at 68.834 91.059 0)
+      (effects (font (size 1.27 1.27)) hide)
+    )
+    (property "Datasheet" "~" (at 68.834 91.059 0)
+      (effects (font (size 1.27 1.27)) hide)
+    )
+    (pin "1")
+    (pin "2")
+    (instances
+      (project "EtherCAT_FUNC"
+        (path "/342eefad-8419-4edc-841f-71a31e56750b/e0fc0fcc-c6e0-408f-913f-bc6bd8418cc7"
+          (reference "R4") (unit 1)
+        )
+        (path "/342eefad-8419-4edc-841f-71a31e56750b"
+          (reference "R8") (unit 1)
+        )
+      )
+      (project "USB2UART"
+        (path "/75368248-08b1-4e75-aab1-d4baf4ebc338"
+          (reference "R1") (unit 1)
+        )
+      )
+      (project "EtherCAT2XXX"
+        (path "/8e0527a1-64cc-4c21-af5a-5910f4c387cc/fa5393d6-c3e4-4b31-a507-98a55f9f6a14"
+          (reference "R23") (unit 1)
+        )
+      )
+    )
+  )
   (symbol (lib_id "power:GND") (at 80.518 64.135 0) (unit 1)
     (in_bom yes) (on_board yes) (dnp no) (fields_autoplaced)
@@
         )
       )
+    )
+  )
+  (symbol (lib_id "power:GND") (at 68.834 107.061 0) (mirror y) (unit 1)
+    (in_bom yes) (on_board yes) (dnp no)
+    (property "Reference" "#PWR033" (at 68.834 113.411 0)
+      (effects (font (size 1.27 1.27)) hide)
+    )
+    (property "Value" "GND" (at 66.802 110.617 0)
+      (effects (font (size 1.27 1.27)) (justify right))
+    )
+    (property "Footprint" "" (at 68.834 107.061 0)
+      (effects (font (size 1.27 1.27)) hide)
+    )
+    (property "Datasheet" "" (at 68.834 107.061 0)
+      (effects (font (size 1.27 1.27)) hide)
+    )
+    (pin "1")
+    (instances
+      (project "EtherCAT_FUNC"
+        (path "/342eefad-8419-4edc-841f-71a31e56750b"
+          (reference "#PWR033") (unit 1)
+        )
+      )
+      (project "USB2UART"
+        (path "/75368248-08b1-4e75-aab1-d4baf4ebc338"
+          (reference "#PWR01") (unit 1)
+        )
+      )
+      (project "ethercat"
+        (path "/e719c6e2-2b94-490a-8084-d00cca2a4437/7cf17e07-07eb-4777-9fca-1fa45a1d7eb7"
+          (reference "#PWR0109") (unit 1)
+        )
+      )
