File: USB_HUB.kicad_sch (KiCad schematic)
At the start: 7 parts, among them U1 SL2.1S, Y1 12M

Commit message: All 0603 version
Parts:
- C1, C3: value 18p -> 20p; footprint Capacitor_SMD:C_0402_1005Metric -> Capacitor_SMD:C_0603_1608Metric
- C2, C4, C5: footprint Capacitor_SMD:C_0402_1005Metric -> Capacitor_SMD:C_0603_1608Metric
Changed lines of the file:
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@@
       (effects (font (size 1.27 1.27)) (justify left))
     )
-    (property "Value" "18p" (at 108.585 92.456 0)
-      (effects (font (size 1.27 1.27)) (justify right))
-    )
-    (property "Footprint" "Capacitor_SMD:C_0402_1005Metric" (at 109.093 90.932 0)
+    (property "Value" "20p" (at 108.585 92.456 0)
+      (effects (font (size 1.27 1.27)) (justify right))
+    )
+    (property "Footprint" "Capacitor_SMD:C_0603_1608Metric" (at 109.093 90.932 0)
       (effects (font (size 1.27 1.27)) hide)
     )
@@
       (effects (font (size 1.27 1.27)))
     )
-    (property "Footprint" "Capacitor_SMD:C_0402_1005Metric" (at 148.209 83.312 0)
+    (property "Footprint" "Capacitor_SMD:C_0603_1608Metric" (at 148.209 83.312 0)
       (effects (font (size 1.27 1.27)) hide)
     )
@@
       (effects (font (size 1.27 1.27)))
     )
-    (property "Footprint" "Capacitor_SMD:C_0402_1005Metric" (at 148.209 86.868 0)
+    (property "Footprint" "Capacitor_SMD:C_0603_1608Metric" (at 148.209 86.868 0)
       (effects (font (size 1.27 1.27)) hide)
     )
@@
       (effects (font (size 1.27 1.27)) (justify right))
     )
-    (property "Footprint" "Capacitor_SMD:C_0402_1005Metric" (at 116.205 114.808 0)
+    (property "Footprint" "Capacitor_SMD:C_0603_1608Metric" (at 116.205 114.808 0)
       (effects (font (size 1.27 1.27)) hide)
     )
@@
       (effects (font (size 1.27 1.27)))
     )
-    (property "Value" "18p" (at 121.031 99.695 90)
-      (effects (font (size 1.27 1.27)))
-    )
-    (property "Footprint" "Capacitor_SMD:C_0402_1005Metric" (at 117.729 98.552 0)
-      (effects (font (size 1.27 1.27)) hide)
-    )
+    (property "Value" "20p" (at 121.031 99.695 90)
+      (effects (font (size 1.27 1.27)))
+    )
+    (property "Footprint" "Capacitor_SMD:C_0603_1608Metric" (at 117.729 98.552 0)
+      (effects (font (size 1.27 1.27)) hide)
+    )
